Commit message: trajectory & context sim succ

File: src/msr_simulation/urdf/puzzlebot.urdf.xacro (robot description, xacro)
@@ -4,4 +4,5 @@
   <link name="base_link">
     <visual>
+      <origin xyz="0 0 0.05" rpy="0 0 0"/>
       <geometry>
         <mesh filename="package://msr_simulation/meshes/chassis1.dae" scale="1 1 1"/>
@@ -15,5 +16,5 @@
     <inertial>
       <mass value="0.8"/>
-      <origin xyz="-0.05 0 0" rpy="0 0 0"/>
+      <origin xyz="-0.05 0 0.05" rpy="0 0 0"/>
       <inertia ixx="0.004" ixy="0" ixz="0" iyy="0.004" iyz="0" izz="0.004"/>
     </inertial>
@@ -39,5 +40,5 @@
     <parent link="base_link"/>
     <child link="left_wheel"/>
-    <origin xyz="0 0.095 0" rpy="0 0 0"/>
+    <origin xyz="0 0.095 0.05" rpy="0 0 0"/>
     <axis xyz="0 1 0"/>
   </joint>
@@ -62,5 +63,5 @@
     <parent link="base_link"/>
     <child link="right_wheel"/>
-    <origin xyz="0 -0.095 0" rpy="0 0 3.1415"/>
+    <origin xyz="0 -0.095 0.05" rpy="0 0 3.1415"/>
     <axis xyz="0 1 0"/>
   </joint>
